File: SCR_PCB/untitled.kicad_sch (KiCad schematic)
At the start: 15 parts, among them Q2 Q_NMOS, U4 SFH617A-1

Commit message: update SRC_PCB
Connections:
- net GATE: now reaches C3.2, C4.2, D10.2 (A), D9.2 (A), Q2.S, R9.2
- net Kathode: now reaches D11.2 (A), D12.2 (A)
- net TRG: now reaches R6.1

Commit message: add SCR PCB
Parts:
- removed D9: D_Zener, symbol Device:D_Zener
- removed Q2: Q_NMOS, symbol Device:Q_NMOS
- added Q1: QM6006D, Package_TO_SOT_SMD:TO-252-2, symbol Transistor_FET:QM6006D
- C3, C4: footprint (none) -> Capacitor_SMD:C_0805_2012Metric
- D10, D11, D12, D7: footprint (none) -> Diode_SMD:D_SMA
- D8: footprint (none) -> LED_SMD:LED_1206_3216Metric
- R10: footprint (none) -> Resistor_THT:R_Axial_DIN0918_L18.0mm_D9.0mm_P22.86mm_Horizontal
- R6: value 1k -> 220R; footprint (none) -> Resistor_SMD:R_0805_2012Metric
- R7, R9: footprint (none) -> Resistor_SMD:R_0805_2012Metric
- R8: footprint (none) -> Resistor_THT:R_Axial_DIN0207_L6.3mm_D2.5mm_P10.16mm_Horizontal
Connections:
- net GATE: now also Q1.3 (S)
- net at C3.1, R9.1, U4.3: now also Q1.1 (G)
- net at R10.2: now also Q1.2 (D)
- net Kathode renamed Anode
