File: DRSSTC_STM32_Controller/MCU.kicad_sch (KiCad schematic)
At the start: 39 parts, among them J13 USB_C_Receptacle_USB2.0_14P, J14 Conn_01x02, J15 Conn_01x02, J16 Conn_01x05, J3 Conn_02x05_Odd_Even, U1 STM32G474RETx

Commit message: update the feedback stage simulation & controller schematic
Other:
- moved on the sheet: C22, C23, C24, C25, C26, C27, C48, C49, C50, C51, D17, D18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

Commit message: update conroller schematics
Parts:
- removed C48, C49: 1u, symbol Device:C
- removed D26: ESDA5V3L, Package_TO_SOT_SMD:SOT-23-3, symbol Power_Protection:ESDA5V3L
- removed D27, D28, D29, D30: D_Zener, symbol Device:D_Zener
- removed J13: USB_C_Receptacle_USB2.0_14P, symbol Connector:USB_C_Receptacle_USB2.0_14P
- removed J16: Conn_01x05, symbol Connector_Generic:Conn_01x05
- removed R76, R77, R78, R79: 220R, Resistor_SMD:R_0805_2012Metric, symbol Device:R
- added C30, C31: 1u, Capacitor_SMD:C_0805_2012Metric, symbol Device:C
- added C63: 1u, symbol Device:C
- added C77, C78: 27p, symbol Device:C
- added D26, D27, D28, D29: YLED1206R, LED_SMD:LED_1206_3216Metric, symbol Device:LED
- added D43, D47, D48, D8: ESDA5V3L, Package_TO_SOT_SMD:SOT-23-3, symbol Power_Protection:ESDA5V3L
- added H1, H2, H3: MountingHole, symbol Mechanical:MountingHole
- added H4: MountingHole_Pad, symbol Mechanical:MountingHole_Pad
- added IC8: PLT237_T10WH, Library:PLT237T10WH, symbol Library:PLT237_T10WH
- added J2, J27: Conn_01x04, symbol Connector_Generic:Conn_01x04
- added R115, R152: 0R, Resistor_SMD:R_0805_2012Metric, symbol Device:R
- added R118, R122, R137, R138, R157, R158, R52, R53, R54, R55: 100R, Resistor_SMD:R_0805_2012Metric, symbol Device:R
- added R153, R154, R159, R160, R161, R162: 22R, Resistor_SMD:R_0805_2012Metric, symbol Device:R
- added R155, R156: 5.1k, Resistor_SMD:R_0805_2012Metric, symbol Device:R
- added R56, R57: 10k, Resistor_SMD:R_0805_2012Metric, symbol Device:R
- added TP1: nrst, symbol Connector:TestPoint
- added U2: PLR237_T10BK, Library:PLR237T10BK, symbol Library:PLR237_T10BK
- added Y1: Crystal, symbol Device:Crystal
- R88, R89, R90, R91: value 1k -> 220R
Connections:
- net +3V3: now also C30.1, C31.1, IC8.2 (VCC), J2.2 (Pin_2), J27.2 (Pin_2), U2.2 (GND)
- net GND: now also C30.2, C31.2, C63.2, C77.2, C78.2, D26.1 (K), D27.1 (K), D28.1 (K), D29.1 (K), D43.3 (A), D47.3 (A), D48.3 (A), D8.3 (A), IC8.3 (GND), J2.1 (Pin_1), J27.1 (Pin_1), R115.1, R152.1, R155.1, R156.1, R56.1, R57.1, U2.3 (VOUT); no longer U1.27 (VSSA)
- net SCL: now reaches U1.10 (PC2)
- net SCL: now also R52.1, R55.1
- net SDA: now reaches U1.11 (PC3)
- net SDA: now also R53.1, R54.1
- net ZCD_-: now reaches U1.12 (PA0)
- net ZCD_+: now reaches U1.13 (PA1)
- net Temp1: now reaches U1.14 (PA2)
- net Temp2: now reaches U1.17 (PA3)
- net 3V3Asense: now reaches U1.18 (PA4)
- net 3V3sense: now reaches U1.19 (PA5)
- net at U1.2 (PC13): now also R90.2
- net Temp3: now reaches U1.20 (PA6)
- net OCD: now reaches U1.21 (PA7)
- net Temp4: now reaches U1.22 (PC4)
- net at U1.23 (PC5): now also R88.2
- net OPAMP+: now reaches U1.24 (PB0)
- net OPAMP_out: now reaches U1.25 (PB1)
- net OPAMP-: now reaches U1.26 (PB2)
- net at U1.28 (VREF+): now also C51.1, C63.1
- net GPIO1: now reaches U1.3 (PC14)
- net GPIO1: now also C47.1, D24.1 (K), R86.1, R56.2
- net Rly_3: now reaches U1.33 (PB11)
- net at U1.34 (PB12): now also R118.1
- net at U1.35 (PB13): now also R122.2
- net at U1.37 (PB15): now also R156.2, R158.2
- net EXT_LED1: now reaches U1.38 (PC6)
- net EXT_LED2: now reaches U1.39 (PC7)
- net GPIO2: now reaches U1.4 (PC15)
- net GPIO2: now also C46.1, D25.1 (K), R87.1, R57.2
- net EXT_LED3: now reaches U1.40 (PC8)
- net EXT_LED4: now reaches U1.41 (PC9)
- net at U1.42 (PA8): now also R137.1
- net at U1.43 (PA9): now also R138.2
- net 12V_EN: now reaches U1.44 (PA10)
- net at U1.45 (PA11): now also R153.1
- net at U1.46 (PA12): now also R154.2
- net at U1.49 (PA13): now also R161.1
- net at U1.5 (PF0): now also C77.1, Y1.1
- net at U1.50 (PA14): now also R162.2
- net at U1.51 (PA15): now also R155.2, R157.2
- net at U1.52 (PC10): now also R159.2
- net UART_RX: now reaches U1.53 (PC11)
- net UART_RX: now also R160.2
- net at U1.54 (PC12): now also R89.2
- net Rly_4: now reaches U1.55 (PD2)
- net Rly_1: now reaches U1.56 (PB3)
- net Rly_2: now reaches U1.57 (PB4)
- net at U1.58 (PB5): now also R91.2
- net FAN1_pwm: now reaches U1.59 (PB6)
- net at U1.6 (PF1): now also C78.1, Y1.2
- net FAN2_pwm: now reaches U1.60 (PB7)
- net FAN3_pwm: now reaches U1.61 (PB8)
- net FAN4_pwm: now reaches U1.62 (PB9)
- net NRST: now reaches U1.7 (PG10)
- net NRST: now also C50.1, TP1.1
- net 12Vsense: now reaches U1.8 (PC0)
- net 24Vsense: now reaches U1.9 (PC1)
- net G1+: now reaches D18.1 (K), J3.3 (Pin_3)
- net G1+: now also R137.2
- net G1-: now reaches D18.2 (K), J3.5 (Pin_5)
- net G1-: now also R138.1
- net G2+: now reaches D17.1 (K), J3.7 (Pin_7)
- net G2+: now also R118.2
- net G2-: now reaches D17.2 (K), J3.9 (Pin_9)
- net G2-: now also R122.1
- net at R90.1: now also D28.2 (A); no longer C51.1
- net at R89.1: now also D27.2 (A); no longer C50.1
- net at R88.1: now also D26.2 (A)
- net at R91.1: now also D29.2 (A)
- net at D31.2 (K): now also J27.4 (Pin_4), R55.2; no longer R90.2
- net at D31.1 (K): now also J27.3 (Pin_3), R54.2; no longer R89.2
- new net: R115.2, U1.27 (VSSA)
- new net: R160.1, U2.1 (VCC)
- new net: D8.2 (K), J2.4 (Pin_4), R52.2
- new net: D8.1 (K), J2.3 (Pin_3), R53.2
- new net Earth_Protective: H4.1, R152.2
- new net SYS_JTCK-SWCLK: D48.1 (K), R162.1
- new net SYS_JTMS-SWDIO: D48.2 (K), R161.2
- new net UART_TX: IC8.1 (VIN), R159.1
- new net USB+: D43.1 (K), R154.1
- new net USB-: D43.2 (K), R153.2
- new net USB_CC1: D47.2 (K), R157.1
- new net USB_CC2: D47.1 (K), R158.1
- no-connect marks 0 -> 1
Other:
- note added: "EXT gate outs"
- note added: "GND to Case (earth) connection"
- note added: "GPIO"
- note added: "MCU Decoupling"
- note added: "SWD"
- note added: "Vbus monitor"
- note added: "fiber"
- note added: "fiber comms"
- note added: "i2c"
- note added: "inducator LEDS"
- note added: "power sequencing"
- note removed: "EXT gate driver"
- note removed: "GPI"
- note removed: "USB"
- moved on the sheet: C22, C23, C24, C25, C26, C27, C46, C47, D17, D18, D23, D24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

Commit message: assign footprints
Parts:
- removed J14, J15: Conn_01x02, symbol Connector_Generic:Conn_01x02
- C23, C25, C26, C27, C30, C31: footprint Capacitor_SMD:C_0805_2012Metric -> Capacitor_SMD:C_0603_1608Metric
- C46, C47, C50, C51, C63, C77, C78: footprint (none) -> Capacitor_SMD:C_0603_1608Metric
- D24, D25: footprint (none) -> Diode_SMD:D_SOD-323F
- H1, H2, H3: footprint (none) -> MountingHole:MountingHole_3.2mm_M3
- H4: footprint (none) -> MountingHole:MountingHole_3.2mm_M3_Pad_Via
- J2, J27: footprint (none) -> Library:4PIN SMD 2.54
- J3: footprint (none) -> Connector_IDC:IDC-Header_2x05_P2.54mm_Vertical
- R115, R118, R122, R137, R138, R152, R153, R154, R155, R156, R157, R158, R159, R160, R161, R162, R52, R53, R54, R55, R56, R57, R86, R87: footprint Resistor_SMD:R_0805_2012Metric -> Resistor_SMD:R_0603_1608Metric
- TP1: footprint (none) -> TestPoint:TestPoint_Pad_2.0x2.0mm
- Y1: footprint (none) -> Crystal:Crystal_SMD_3225-4Pin_3.2x2.5mm
Connections:
- net GPIO_1: now reaches D23.2 (K), R86.2
- net GPIO_2: now reaches D23.1 (K), R87.2
