File: DRSSTC_STM32_Controller/MCU.kicad_sch (KiCad schematic)
At the start: 69 parts, among them IC8 PLT237_T10WH, J2 Conn_01x04, J27 Conn_01x04, J3 Conn_02x05_Odd_Even, U1 STM32G474RETx, U2 PLR237_T10BK, Y1 Crystal

Commit message: re-do the layout
Changed lines of the file:
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@@
 	(text "fiber comms\n"
 		(exclude_from_sim no)
-		(at 84.582 43.942 0)
+		(at 73.66 36.576 0)
 		(effects
 			(font

Commit message: start routing
Parts:
- removed R152: 0R, Resistor_SMD:R_0603_1608Metric, symbol Device:R
Connections:
- net Earth_Protective: no longer H4.1
- net GND: now also H4.1
Changed lines of the file:
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@@
 	)
 	(junction
-		(at 241.3 254)
-		(diameter 0)
-		(color 0 0 0 0)
-	)
-	(junction
 		(at 344.17 107.95)
 		(diameter 0)
@@
 	(wire
 		(pts
-			(xy 241.3 252.73) (xy 241.3 254)
+			(xy 241.3 252.73) (xy 241.3 264.16)
 		)
 		(stroke
@@
 	(wire
 		(pts
-			(xy 241.3 262.89) (xy 241.3 264.16)
-		)
-		(stroke
-			(width 0)
-			(type default)
-		)
-	)
-	(wire
-		(pts
 			(xy 275.59 173.99) (xy 278.13 173.99)
 		)
@@
 	(wire
 		(pts
-			(xy 241.3 254) (xy 241.3 255.27)
-		)
-		(stroke
-			(width 0)
-			(type default)
-		)
-	)
-	(wire
-		(pts
 			(xy 307.34 133.35) (xy 309.88 133.35)
 		)
@@
 	(wire
 		(pts
-			(xy 241.3 254) (xy 260.35 254)
-		)
-		(stroke
-			(width 0)
-			(type default)
-		)
-	)
-	(wire
-		(pts
 			(xy 232.41 110.49) (xy 227.33 110.49)
 		)
@@
 	(wire
 		(pts
-			(xy 260.35 255.27) (xy 260.35 254)
+			(xy 269.24 255.27) (xy 269.24 254)
 		)
 		(stroke
@@
 	)
 	(symbol
-		(lib_id "Device:R")
-		(at 241.3 259.08 0)
-		(mirror x)
-		(unit 1)
-		(body_style 1)
-		(exclude_from_sim no)
-		(in_bom yes)
-		(on_board yes)
-		(in_pos_files yes)
-		(dnp no)
-		(property "Reference" "R152"
-			(at 245.11 260.35 0)
-			(show_name no)
-			(do_not_autoplace no)
-			(effects
-				(font
-					(size 1.27 1.27)
-				)
-			)
-		)
-		(property "Value" "0R"
-			(at 245.11 257.81 0)
-			(show_name no)
-			(do_not_autoplace no)
-			(effects
-				(font
-					(size 1.27 1.27)
-				)
-			)
-		)
-		(property "Footprint" "Resistor_SMD:R_0603_1608Metric"
-			(at 239.522 259.08 90)
-			(hide yes)
-			(show_name no)
-			(do_not_autoplace no)
-			(effects
-				(font
-					(size 1.27 1.27)
-				)
-			)
-		)
-		(property "Datasheet" ""
-			(at 241.3 259.08 0)
-			(hide yes)
-			(show_name no)
-			(do_not_autoplace no)
-			(effects
-				(font
-					(size 1.27 1.27)
-				)
-			)
-		)
-		(property "Description" "Resistor"
-			(at 241.3 259.08 0)
-			(hide yes)
-			(show_name no)
-			(do_not_autoplace no)
-			(effects
-				(font
-					(size 1.27 1.27)
-				)
-			)
-		)
-		(pin "1"
-		)
-		(pin "2"
-		)
-		(instances
-			(project "DRSSTC_STM32_Controller"
-				(path "/1b08b5a8-62c7-4a0a-af72-03cffe829476/20c2d3c1-5581-4763-931a-12a331abb72a"
-					(reference "R152")
-					(unit 1)
-				)
-			)
-		)
-	)
-	(symbol
 		(lib_id "Device:C")
 		(at 113.03 99.06 0)
@@
 	(symbol
 		(lib_id "power:Earth_Protective")
-		(at 260.35 255.27 0)
+		(at 269.24 255.27 0)
 		(unit 1)
 		(body_style 1)
@@
 		(fields_autoplaced yes)
 		(property "Reference" "#PWR018"
-			(at 260.35 265.43 0)
+			(at 269.24 265.43 0)
 			(hide yes)
 			(show_name no)
@@
 		)
 		(property "Value" "Earth_Protective"
-			(at 260.35 264.16 0)
+			(at 269.24 264.16 0)
 			(show_name no)
 			(do_not_autoplace no)
@@
 		)
 		(property "Footprint" ""
-			(at 260.35 257.81 0)
+			(at 269.24 257.81 0)
 			(hide yes)
 			(show_name no)
@@
 		)
 		(property "Datasheet" ""
-			(at 260.35 257.81 0)
+			(at 269.24 257.81 0)
 			(hide yes)
 			(show_name no)
@@
 		)
 		(property "Description" "Power symbol creates a global label with name \"Earth_Protective\""
-			(at 260.35 255.27 0)
+			(at 269.24 255.27 0)
 			(hide yes)
 			(show_name no)

Commit message: finalize the controller design
Parts:
- removed H1, H2, H3: MountingHole, MountingHole:MountingHole_3.2mm_M3, symbol Mechanical:MountingHole
- added D50: ESDA5V3L, Package_TO_SOT_SMD:SOT-23-3, symbol Power_Protection:ESDA5V3L
- added H5, H6, H7: MountingHole_Pad, MountingHole:MountingHole_3.2mm_M3_Pad_Via, symbol Mechanical:MountingHole_Pad
- added R69, R77: 4k7, Resistor_SMD:R_0603_1608Metric, symbol Device:R
Connections:
- net +3V3: now also R69.1, R77.1
- net GND: now also D50.3 (A), H5.1, H6.1, H7.1
- net GPIO_2: now also D50.1 (K); no longer D23.1 (K)
- net SCL: now also R77.2
- net SDA: now also R69.2
- net USB_N: now reaches R153.1, U1.45 (PA11)
- net USB_P: now reaches R154.2, U1.46 (PA12)
- no-connect marks 1 -> 3
