File: DRSSTC_STM32_Controller/DRSSTC_STM32_Controller.kicad_pcb (KiCad board)
At the start: 4 copper layers, 100 x 100 mm, 319 parts, among them IC1 UCC27282DR, IC2 UCC27282DR, IC3 UCC27282DR, IC4 UCC27282DR, IC5 SN74LVC14ADR, IC6 SN74LVC11ADR, IC7 SN74LVC11ADR, IC8 PLT237_T10WH, J1 Conn_01x04, J10 Conn_01x04, J11 Conn_01x04, J12 Conn_01x10, J13 USB_C_Receptacle_USB2.0_14P, J14 Conn_01x10, J16 Conn_01x04, J17 Conn_01x10, J2 Conn_01x04, J27 Conn_01x04, J28 Screw_Terminal_01x02, J29 Screw_Terminal_01x02, J3 Conn_02x05_Odd_Even, J30 Screw_Terminal_01x02, J31 Screw_Terminal_01x02, J32 Screw_Terminal_01x02, J33 Screw_Terminal_01x02, J4 Screw_Terminal_01x02, J42 Screw_Terminal_01x02, J5 Conn_Coaxial, J6 Conn_Coaxial, J7 Conn_01x04, Q1 QM6006D, Q10 2N7002, Q11 2N7002, Q12 2N7002, Q13 2N7002, Q14 2N7002, Q15 QM6006D, Q16 QM6006D, Q17 QM6006D, Q18 QM6006D, Q19 2N7002, Q2 QM6006D, Q20 2N7002, Q3 QM6006D, Q4 QM6006D, Q5 2N7002, Q6 2N7002, Q7 2N7002, Q8 2N7002, Q9 2N7002, U1 STM32G474RETx, U2 PLR237_T10BK, U3 LF15_TO252, U4 TPS54560BDDA, U7 LV2842XLVDDCR, Y1 Crystal

Commit message: refine conroller layout
Parts:
- J16: moved to F.Cu
- moved J30 222.6 mm to (353.7, 106.5)
- moved J33 205.9 mm to (313.1, 125.9), turned to 90 degrees
- moved J32 199.0 mm to (313.1, 97.3), turned to -90 degrees
- moved J17 195.7 mm to (291.0, 85.0), turned to 0 degrees
- moved R139 185.8 mm to (274.3, 128.6), turned to 180 degrees
- moved R133 181.6 mm to (274.3, 124.8)
- moved J29 176.2 mm to (287.3, 133.4)
- moved J16 175.6 mm to (251.8, 124.9)
- moved R136 175.3 mm to (284.9, 126.0), turned to 180 degrees
- moved J28 171.7 mm to (252.0, 157.4)
- moved R120 171.4 mm to (284.9, 128.1), turned to 180 degrees
- moved R119 171.3 mm to (284.9, 124.2)
- moved C80 171.2 mm to (284.9, 120.3), turned to 180 degrees
- moved J14 168.2 mm to (254.0, 72.6), turned to 0 degrees
- moved C67 167.8 mm to (284.9, 129.9), turned to 180 degrees
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Routing:
- net Net-(IC5-3Y): track 0.00 -> 36.8 mm, vias 0 -> 3
- net /MCU and comms/G1-: track 0.00 -> 32.3 mm, vias 0 -> 1
- net Net-(IC5-4Y): track 0.00 -> 31.0 mm, vias 0 -> 3
- net Net-(IC5-2Y): track 0.00 -> 30.4 mm, vias 0 -> 3
- net /MCU and comms/G2+: track 0.00 -> 26.2 mm, vias 0 -> 2
- net Net-(IC5-1Y): track 0.00 -> 25.5 mm, vias 0 -> 3
- net /MCU and comms/G2-: track 0.00 -> 19.9 mm, vias 0 -> 2
- net /MCU and comms/G1+: track 0.00 -> 13.6 mm, vias 0 -> 2
- net Net-(IC1-LI): track 0.00 -> 10.5 mm, vias 0 -> 1
- net Net-(IC6-3Y): track 0.00 -> 3.01 mm
- net Net-(IC7-3Y): track 0.00 -> 2.75 mm
- net Net-(IC6-2Y): track 0.00 -> 1.78 mm
- net Net-(IC7-2Y): track 0.00 -> 1.73 mm
Other:
- outline, holes or cut-outs redrawn

Commit message: start cintrollenr routing
Parts:
- removed R69: 10k, Resistor_SMD:R_0603_1608Metric
- C6, C7: footprint Capacitor_SMD:C_0201_0603Metric -> Capacitor_SMD:C_0603_1608Metric
- R102, R132, R47, R92: footprint Resistor_THT:R_Axial_DIN0309_L9.0mm_D3.2mm_P12.70mm_Horizontal -> Resistor_SMD:R_2512_6332Metric
- R67: value 10k -> 5k1
- moved R54 69.2 mm to (243.9, 159.3)
- moved R52 69.2 mm to (248.4, 154.0)
- moved R53 69.2 mm to (248.4, 159.3)
- moved D31 69.2 mm to (243.5, 156.7)
- moved D8 69.2 mm to (247.9, 156.6)
- moved R55 69.2 mm to (243.9, 154.1)
- moved J30 64.2 mm to (291.2, 91.9), turned to 0 degrees
- moved J2 63.6 mm to (252.1, 150.1)
- moved J27 63.3 mm to (251.9, 158.9)
- moved J1 36.8 mm to (325.0, 159.2), turned to 180 degrees
- moved D25 32.5 mm to (291.0, 69.1), turned to 180 degrees
- moved R87 29.4 mm to (291.1, 70.8)
- moved C46 29.3 mm to (294.3, 70.8)
- moved R57 29.3 mm to (294.3, 69.2)
- moved D23 29.0 mm to (294.3, 73.6), turned to -90 degrees
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Routing:
- net /MCU and comms/Rly_4: track 0.00 -> 118.4 mm, vias 0 -> 4
- net GND: track 0.00 -> 107.6 mm, vias 0 -> 262
- net /MCU and comms/Rly_2: track 0.00 -> 106.1 mm, vias 0 -> 4
- net /MCU and comms/Rly_1: track 0.00 -> 100.8 mm, vias 0 -> 4
- net /MCU and comms/EXT_LED1: track 0.00 -> 98.0 mm, vias 0 -> 2
- net /MCU and comms/EXT_LED2: track 0.00 -> 92.4 mm, vias 0 -> 2
- net /MCU and comms/EXT_LED3: track 0.00 -> 84.6 mm, vias 0 -> 2
- net /MCU and comms/Rly_3: track 0.00 -> 80.1 mm, vias 0 -> 2
- net /MCU and comms/EXT_LED4: track 0.00 -> 79.6 mm, vias 0 -> 2
- net /MCU and comms/G1-: track 32.3 -> 90.9 mm, vias 1 -> 6
- net /MCU and comms/G2-: track 19.9 -> 78.3 mm, vias 2 -> 7
- net /MCU and comms/G2+: track 26.2 -> 83.7 mm, vias 2 -> 7
- net /MCU and comms/GPIO2: track 0.00 -> 56.7 mm, vias 0 -> 4
- net /MCU and comms/G1+: track 13.6 -> 68.9 mm, vias 2 -> 7
- net Net-(IC3-HI): track 0.00 -> 51.2 mm, vias 0 -> 3
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- added copper zone on B.Cu, net GND
- added copper zone on F.Cu, net GND
- added copper zone on In1.Cu, net GND
