File: DRSSTC_STM32_Controller/DRSSTC_STM32_Controller.kicad_pcb (KiCad board)
At the start: 4 copper layers, 100 x 100 mm, 318 parts, among them IC1 UCC27282DR, IC2 UCC27282DR, IC3 UCC27282DR, IC4 UCC27282DR, IC5 SN74LVC14ADR, IC6 SN74LVC11ADR, IC7 SN74LVC11ADR, IC8 PLT237_T10WH, J1 Conn_01x04, J10 Conn_01x04, J11 Conn_01x04, J12 Conn_01x10, J13 USB_C_Receptacle_USB2.0_14P, J14 Conn_01x10, J16 Conn_01x04, J17 Conn_01x10, J2 Conn_01x04, J27 Conn_01x04, J28 Screw_Terminal_01x02, J29 Screw_Terminal_01x02, J3 Conn_02x05_Odd_Even, J30 Screw_Terminal_01x02, J31 Screw_Terminal_01x02, J32 Screw_Terminal_01x02, J33 Screw_Terminal_01x02, J4 Screw_Terminal_01x02, J42 Screw_Terminal_01x02, J5 Conn_Coaxial, J6 Conn_Coaxial, J7 Conn_01x04, Q1 QM6006D, Q10 2N7002, Q11 2N7002, Q12 2N7002, Q13 2N7002, Q14 2N7002, Q15 QM6006D, Q16 QM6006D, Q17 QM6006D, Q18 QM6006D, Q19 2N7002, Q2 QM6006D, Q20 2N7002, Q3 QM6006D, Q4 QM6006D, Q5 2N7002, Q6 2N7002, Q7 2N7002, Q8 2N7002, Q9 2N7002, U1 STM32G474RETx, U2 PLR237_T10BK, U3 LF15_TO252, U4 TPS54560BDDA, U7 LV2842XLVDDCR, Y1 Crystal

Commit message: re-do the layout
Parts:
- C1, C12, C13, C2, C3: moved to B.Cu
- moved D26 230.7 mm to (412.5, 295.2)
- moved D29 230.7 mm to (412.5, 300.0)
- moved D27 230.7 mm to (412.5, 297.6)
- moved D28 230.7 mm to (412.5, 302.4)
- moved R89 230.7 mm to (408.4, 297.6)
- moved R88 230.7 mm to (408.4, 295.2)
- moved R91 230.7 mm to (408.4, 300.0)
- moved R90 230.7 mm to (408.4, 302.4)
- moved R47 222.5 mm to (251.0, 279.6), turned to -90 degrees
- moved R46 221.9 mm to (247.4, 278.1), turned to 0 degrees
- moved R45 218.9 mm to (247.5, 276.5), turned to 180 degrees
- moved R92 218.7 mm to (258.0, 279.6), turned to -90 degrees
- moved C33 217.6 mm to (206.4, 271.1), turned to -90 degrees
- moved R101 217.6 mm to (254.5, 278.1), turned to 0 degrees
- moved D38 216.8 mm to (153.3, 290.9), turned to -90 degrees
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Routing:
- net /MCU and comms/Rly_4: track 118.4 -> 1.00 mm, vias 4 -> 1
- net /MCU and comms/Rly_2: track 106.1 -> 0.77 mm, vias 4 -> 1
- net /MCU and comms/Rly_1: track 100.8 -> 0.86 mm, vias 4 -> 1
- net /MCU and comms/EXT_LED1: track 98.0 -> 0.97 mm, vias 2 -> 1
- net /MCU and comms/EXT_LED2: track 92.4 -> 1.19 mm, vias 2 -> 1
- net /MCU and comms/EXT_LED3: track 84.6 -> 1.22 mm, vias 2 -> 1
- net /MCU and comms/Rly_3: track 80.1 -> 0.87 mm, vias 2 -> 1
- net /MCU and comms/EXT_LED4: track 79.6 -> 1.38 mm, vias 2 -> 1
- net /MCU and comms/G2-: track 78.3 -> 9.27 mm, vias 7 -> 3
- net /MCU and comms/G2+: track 83.7 -> 14.7 mm, vias 7 -> 4
- net /MCU and comms/G1-: track 90.9 -> 25.7 mm, vias 6 -> 2
- net Net-(IC3-HI): track 51.2 -> 5.44 mm
- net /Feedback & sensing/Temp1: track 50.8 -> 5.61 mm, vias 4 -> 2
- net /Feedback & sensing/Temp4: track 51.0 -> 5.95 mm, vias 5 -> 2
- net /MCU and comms/G1+: track 68.9 -> 24.1 mm, vias 7 -> 3
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Other:
- board size 100 x 100 mm -> 100 x 137.5 mm

Commit message: start routing
Parts:
- removed C74, C8: 2.2u, Capacitor_THT:C_Axial_L12.0mm_D7.5mm_P15.00mm_Horizontal
- removed C75, C9: 1u, Capacitor_THT:C_Axial_L12.0mm_D7.5mm_P15.00mm_Horizontal
- removed J28, J29, J30, J31: Screw_Terminal_01x02, TerminalBlock_MetzConnect:TerminalBlock_MetzConnect_Type094_RT03502HBLU_1x02_P5.00mm_Horizontal
- removed JP8, JP9: SolderJumper_2_Open, Jumper:SolderJumper-2_P1.3mm_Open_RoundedPad1.0x1.5mm
- removed R126, R42: 100R, Resistor_THT:R_Axial_DIN0309_L9.0mm_D3.2mm_P12.70mm_Horizontal
- removed R152: 0R, Resistor_SMD:R_0603_1608Metric
- C28, C29, C37, C38, C48, C70, C71, C72, C73, D2, D3, D47, F1, FL1, JP4, JP7, L2, R76: moved to B.Cu
- IC8, U2: moved to F.Cu
- moved D28 250.6 mm to (263.3, 101.0), turned to -45 degrees
- moved D29 249.6 mm to (266.3, 97.7), turned to -45 degrees
- moved D27 248.0 mm to (268.1, 96.0), turned to -45 degrees
- moved R90 244.0 mm to (266.4, 104.0), turned to -45 degrees
- moved R91 243.0 mm to (269.3, 100.8), turned to -45 degrees
- moved R89 241.4 mm to (271.1, 99.0), turned to -45 degrees
- moved D2 214.7 mm to (324.9, 141.0), turned to -90 degrees
- moved R99 204.6 mm to (241.0, 100.7), turned to 90 degrees
- moved R88 204.4 mm to (279.4, 136.6), turned to 90 degrees
- moved D26 203.9 mm to (279.4, 140.7), turned to 90 degrees
- moved R98 201.8 mm to (237.2, 100.7), turned to 90 degrees
- moved C55 198.5 mm to (248.8, 106.8), turned to 180 degrees
- moved C57 197.6 mm to (249.8, 101.8)
- moved D38 197.3 mm to (248.5, 118.1), turned to 0 degrees
- moved R94 197.1 mm to (252.1, 105.9)
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Connections:
- C45 pad 2: Net-(IC1-HS) -> /GDT_driver/GDT1+
- C68 pad 2: Net-(IC3-HS) -> /GDT_driver/GDT2+
- D2 pad 1: Net-(IC1-HS) -> /GDT_driver/GDT1+
- D3 pad 1: Net-(IC3-HS) -> /GDT_driver/GDT2+
- H4 pad 1: Earth_Protective -> GND
- IC1 pad 4: Net-(IC1-HS) -> /GDT_driver/GDT1+
- IC3 pad 4: Net-(IC3-HS) -> /GDT_driver/GDT2+
- Q1 pad 3: Net-(IC1-HS) -> /GDT_driver/GDT1+
- Q15 pad 3: Net-(IC3-HS) -> /GDT_driver/GDT2+
- Q16 pad 2: Net-(IC3-HS) -> /GDT_driver/GDT2+
- Q2 pad 2: Net-(IC1-HS) -> /GDT_driver/GDT1+
- R97 pad 2: Net-(R97-Pad2) -> Net-(R95-Pad2)
- R99 pad 1: Net-(R97-Pad2) -> Net-(R95-Pad2)
Routing:
- net GND: track 106.6 -> 397.8 mm, vias 218 -> 194
- net /Feedback & sensing/OPAMP+: track 0.00 -> 73.9 mm, vias 0 -> 2
- net /MCU and comms/GPIO2: track 15.1 -> 82.3 mm, vias 0 -> 3
- net /MCU and comms/UART_TX: track 0.00 -> 66.7 mm
- net /Feedback & sensing/OPAMP-: track 0.00 -> 63.1 mm, vias 0 -> 2
- net /MCU and comms/Rly_1: track 0.86 -> 59.1 mm, vias 1 -> 2
- net Net-(U1-PB15): track 1.60 -> 57.3 mm
- net /MCU and comms/12V_EN: track 2.69 -> 57.8 mm, vias 0 -> 1
- net /MCU and comms/G2-: track 9.27 -> 63.4 mm
- net /Feedback & sensing/OPAMP_out: track 0.00 -> 53.8 mm, vias 0 -> 2
- net /MCU and comms/Rly_2: track 0.77 -> 52.7 mm, vias 1 -> 2
- net /MCU and comms/SDA: track 5.13 -> 56.8 mm
- net /MCU and comms/EXT_LED4: track 1.38 -> 51.7 mm, vias 1 -> 0
- net /MCU and comms/Rly_3: track 0.87 -> 50.7 mm, vias 1 -> 2
- net /Feedback & sensing/12Vsens: track 8.51 -> 56.6 mm, vias 1 -> 0
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- added copper zone on B.Cu, net +12V
- added copper zone on F.Cu, net +12V
- added copper zone on B.Cu, net +24V
- added copper zone on F.Cu, net +24V
- added copper zone on B.Cu, net +3V3
- added copper zone on F.Cu, net +3V3
- added copper zone on In2.Cu, net GND
- added copper zone on B.Cu, net Net-(D11-K)
- added copper zone on F.Cu, net Net-(D11-K)
- added copper zone on F.Cu, net Net-(D32-K)
- added copper zone on F.Cu, net Net-(U3-VI)
- added copper zone on F.Cu, net VDDA
Other:
- board size 100 x 137.5 mm -> 100 x 100 mm
