File: DRSSTC_STM32_Controller/Feedback & sense.kicad_sch (KiCad schematic)
At the start: 66 parts

Commit message: start routing
Connections:
- net at R97.2, R99.1: now also R95.2, R98.1
Changed lines of the file:
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@@
+	)
+	(junction
+		(at 140.97 66.04)
+		(diameter 0)
+		(color 0 0 0 0)
 	)
 	(junction
@@
 	(junction
 		(at 165.1 209.55)
+		(diameter 0)
+		(color 0 0 0 0)
+	)
+	(junction
+		(at 133.35 66.04)
 		(diameter 0)
 		(color 0 0 0 0)
@@
 	(wire
 		(pts
+			(xy 133.35 66.04) (xy 133.35 66.2654)
+		)
+		(stroke
+			(width 0)
+			(type default)
+		)
+	)
+	(wire
+		(pts
 			(xy 66.04 115.57) (xy 66.04 110.49)
 		)
@@
 	(wire
 		(pts
-			(xy 133.35 64.77) (xy 133.35 66.2654)
+			(xy 133.35 64.77) (xy 133.35 66.04)
 		)
 		(stroke
@@
 		)
 		(stroke
+			(width 0)
+			(type default)
+		)
+	)
+	(wire
+		(pts
+			(xy 133.35 66.04) (xy 140.97 66.04)
+		)
+		(stroke
