File: DRSSTC_STM32_Controller/untitled.kicad_sch (KiCad schematic)
At the start: 46 parts, among them U3 LF15_TO252, U4 TPS54560BDDA, U7 LV2842XLVDDCR

Commit message: finalize the controller design
Changed lines of the file:
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@@
 	(text "3V3"
 		(exclude_from_sim no)
-		(at 200.914 17.526 0)
+		(at 216.154 26.924 0)
 		(effects
 			(font
